File: Ball40.kicad_pcb (KiCad board)
At the start: 2 copper layers, 82 parts, among them J1 Conn_01x08_Male, J2 USB_C_Receptacle_USB2.0, SW1 SW_Push, U1 SRV05-4, U2 ATmega32U4-AU, Y1 16MHz

Commit message: generated gerbers
Parts:
- moved R3 4.28 mm to (139.9, 130.2)
- moved C3 4.28 mm to (136.7, 112.8)
- moved R6 4.28 mm to (117.7, 130.4)
- moved U2 4.28 mm to (126.6, 121.3)
- moved R5 4.28 mm to (132.5, 109.6)
- moved R4 4.28 mm to (133.9, 111.0)
- turned J1 to 350 degrees
Connections:
- U2 pad 21: Net-(U2-Pad21) -> COL5
- U2 pad 22: Net-(U2-Pad22) -> COL6
- U2 pad 25: Net-(U2-Pad25) -> COL7
- U2 pad 26: Net-(U2-Pad26) -> COL8
- U2 pad 27: Net-(U2-Pad27) -> COL9
- U2 pad 28: Net-(U2-Pad28) -> COL4
- U2 pad 29: Net-(U2-Pad29) -> COL3
- U2 pad 30: Net-(U2-Pad30) -> COL2
- U2 pad 31: Net-(U2-Pad31) -> COL1
- U2 pad 32: Net-(U2-Pad32) -> COL0
Routing:
- net ROW2: track 0.00 -> 316.7 mm, vias 0 -> 2
- net ROW1: track 0.00 -> 306.4 mm, vias 0 -> 2
- net ROW0: track 0.00 -> 273.5 mm, vias 0 -> 2
- net COL9: track 0.00 -> 249.3 mm, vias 0 -> 3
- net COL8: track 0.00 -> 233.1 mm, vias 0 -> 3
- net GND: track 0.00 -> 228.1 mm, vias 0 -> 12
- net COL0: track 0.00 -> 219.1 mm, vias 0 -> 3
- net COL7: track 0.00 -> 215.8 mm, vias 0 -> 3
- net COL1: track 0.00 -> 193.1 mm, vias 0 -> 3
- net COL6: track 0.00 -> 180.2 mm, vias 0 -> 1
- net COL2: track 0.00 -> 174.1 mm, vias 0 -> 3
- net +5V: track 0.00 -> 155.2 mm, vias 0 -> 7
- net COL5: track 0.00 -> 148.6 mm, vias 0 -> 3
- net COL3: track 0.00 -> 144.6 mm, vias 0 -> 3
- net COL4: track 0.00 -> 126.4 mm, vias 0 -> 3
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Other:
- board outline added: 266.7 x 111.8 mm
